File: PCB/RevExpansionHub.kicad_sch (KiCad schematic)
At the start: 88 parts, among them J14 Conn_01x03_Male, J15 JTAG Connector, J20 Servo Connector, J5 Digital 6,7, J6 Digital 4,5, J7 Digital 2,3, J8 Digital 0,1, Q1 Q_NPN_EBC, Q10 N32, Q11 N32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

Commit message: schematic update
Connections:
- net at R31.1: now also U?.104 (PL4); no longer U?.105 (PL3)
- net at R33.1: now also U?.105 (PL3); no longer U?.106 (PL2)
- net at R29.1: no longer U?.104 (PL4)
- net at R35.1: now also U?.106 (PL2)
Changed lines of the file:
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@@
+    (stroke (width 0) (type default))
+  )
+  (wire (pts (xy 796.29 607.06) (xy 701.04 607.06))
     (stroke (width 0) (type default))
   )
@@
     (stroke (width 0) (type default))
   )
+  (wire (pts (xy 514.35 252.73) (xy 514.35 322.58))
+    (stroke (width 0) (type default))
+  )
   (wire (pts (xy 767.08 582.93) (xy 767.08 586.74))
     (stroke (width 0) (type default))
@@
     (stroke (width 0) (type default))
   )
+  (wire (pts (xy 712.47 576.58) (xy 796.29 576.58))
+    (stroke (width 0) (type default))
+  )
   (wire (pts (xy 796.29 539.75) (xy 796.29 553.72))
     (stroke (width 0) (type default))
@@
     (stroke (width 0) (type default))
   )
-  (wire (pts (xy 715.01 576.58) (xy 796.29 576.58))
-    (stroke (width 0) (type default))
-  )
   (wire (pts (xy 807.72 694.69) (xy 807.72 664.21))
     (stroke (width 0) (type default))
@@
     (stroke (width 0) (type default))
   )
-  (wire (pts (xy 718.82 539.75) (xy 718.82 285.75))
+  (wire (pts (xy 712.47 255.27) (xy 712.47 576.58))
     (stroke (width 0) (type default))
   )
@@
     (stroke (width 0) (type default))
   )
-  (wire (pts (xy 715.01 288.29) (xy 715.01 576.58))
-    (stroke (width 0) (type default))
-  )
   (wire (pts (xy 370.84 593.09) (xy 370.84 598.17))
     (stroke (width 0) (type default))
   )
-  (wire (pts (xy 519.43 322.58) (xy 519.43 283.21))
+  (wire (pts (xy 519.43 259.08) (xy 519.43 322.58))
     (stroke (width 0) (type default))
   )
@@
     (stroke (width 0) (type default))
   )
+  (wire (pts (xy 717.55 259.08) (xy 717.55 539.75))
+    (stroke (width 0) (type default))
+  )
   (wire (pts (xy 726.44 280.67) (xy 726.44 469.9))
     (stroke (width 0) (type default))
@@
     (stroke (width 0) (type default))
   )
-  (wire (pts (xy 509.27 322.58) (xy 509.27 293.37))
+  (wire (pts (xy 509.27 322.58) (xy 509.27 247.65))
     (stroke (width 0) (type default))
   )
@@
     (stroke (width 0) (type default))
   )
-  (wire (pts (xy 511.81 290.83) (xy 511.81 322.58))
+  (wire (pts (xy 511.81 250.19) (xy 511.81 322.58))
     (stroke (width 0) (type default))
   )
@@
     (stroke (width 0) (type default))
   )
-  (wire (pts (xy 519.43 283.21) (xy 722.63 283.21))
-    (stroke (width 0) (type default))
-  )
   (wire (pts (xy 383.54 586.74) (xy 383.54 584.2))
     (stroke (width 0) (type default))
@@
     (stroke (width 0) (type default))
   )
+  (wire (pts (xy 516.89 255.27) (xy 712.47 255.27))
+    (stroke (width 0) (type default))
+  )
   (wire (pts (xy 803.91 621.03) (xy 816.61 621.03))
     (stroke (width 0) (type default))
@@
     (stroke (width 0) (type default))
   )
-  (wire (pts (xy 796.29 539.75) (xy 718.82 539.75))
-    (stroke (width 0) (type default))
-  )
   (wire (pts (xy 636.27 400.05) (xy 670.56 400.05))
     (stroke (width 0) (type default))
@@
     (stroke (width 0) (type default))
   )
-  (wire (pts (xy 722.63 283.21) (xy 722.63 505.46))
-    (stroke (width 0) (type default))
-  )
   (wire (pts (xy 692.15 669.29) (xy 692.15 299.72))
     (stroke (width 0) (type default))
@@
     (stroke (width 0) (type default))
   )
-  (wire (pts (xy 509.27 293.37) (xy 704.85 293.37))
+  (wire (pts (xy 509.27 247.65) (xy 704.85 247.65))
     (stroke (width 0) (type default))
   )
@@
     (stroke (width 0) (type default))
   )
-  (wire (pts (xy 708.66 290.83) (xy 511.81 290.83))
+  (wire (pts (xy 708.66 250.19) (xy 511.81 250.19))
     (stroke (width 0) (type default))
   )
@@
     (stroke (width 0) (type default))
   )
+  (wire (pts (xy 717.55 539.75) (xy 796.29 539.75))
+    (stroke (width 0) (type default))
+  )
   (wire (pts (xy 767.08 515.62) (xy 767.08 519.43))
     (stroke (width 0) (type default))
@@
     (stroke (width 0) (type default))
   )
+  (wire (pts (xy 701.04 607.06) (xy 701.04 252.73))
+    (stroke (width 0) (type default))
+  )
   (wire (pts (xy 767.08 549.91) (xy 767.08 553.72))
     (stroke (width 0) (type default))
@@
     (stroke (width 0) (type default))
   )
-  (wire (pts (xy 704.85 293.37) (xy 704.85 678.18))
+  (wire (pts (xy 704.85 247.65) (xy 704.85 678.18))
+    (stroke (width 0) (type default))
+  )
+  (wire (pts (xy 701.04 252.73) (xy 514.35 252.73))
     (stroke (width 0) (type default))
   )
@@
     (stroke (width 0) (type default))
   )
-  (wire (pts (xy 718.82 285.75) (xy 516.89 285.75))
-    (stroke (width 0) (type default))
-  )
   (wire (pts (xy 642.62 666.75) (xy 373.38 666.75))
     (stroke (width 0) (type default))
@@
     (stroke (width 0) (type default))
   )
-  (wire (pts (xy 516.89 285.75) (xy 516.89 322.58))
-    (stroke (width 0) (type default))
-  )
-  (wire (pts (xy 708.66 643.89) (xy 708.66 290.83))
+  (wire (pts (xy 708.66 643.89) (xy 708.66 250.19))
     (stroke (width 0) (type default))
   )
@@
     (stroke (width 0) (type default))
   )
-  (wire (pts (xy 514.35 322.58) (xy 514.35 288.29))
-    (stroke (width 0) (type default))
-  )
-  (wire (pts (xy 514.35 288.29) (xy 715.01 288.29))
-    (stroke (width 0) (type default))
-  )
   (wire (pts (xy 426.72 469.9) (xy 414.02 469.9))
     (stroke (width 0) (type default))
@@
     (stroke (width 0) (type default))
   )
+  (wire (pts (xy 519.43 259.08) (xy 717.55 259.08))
+    (stroke (width 0) (type default))
+  )
   (wire (pts (xy 358.14 718.82) (xy 358.14 720.09))
     (stroke (width 0) (type default))
@@
     (stroke (width 0) (type default))
   )
+  (wire (pts (xy 516.89 255.27) (xy 516.89 322.58))
+    (stroke (width 0) (type default))
+  )
